File: Charlie/charlie.brd (EAGLE design)
At the start: 181.4 x 25.4 mm, 28 parts

Commit message: add proper board file, and add mosfet for reverse battery safety
Parts:
- added Q1: BSA223SP, transistor-fet:SC75_INFINEON
Connections:
- new net N$7: BAT1.1
- net 2.8V: now also Q1.3; no longer BAT1.1
- net GND: now also Q1.1
Routing:
- net 2.8V: track 31.0 -> 27.6 mm
Changed lines of the file:
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@@
 <?xml version="1.0" encoding="utf-8"?>
 <!DOCTYPE eagle SYSTEM "eagle.dtd">
-<eagle version="6.0">
+<eagle version="6.4">
 <drawing>
 <settings>
@@
 <layer number="144" name="Drill_legend" color="7" fill="1" visible="no" active="yes"/>
 <layer number="151" name="HeatSink" color="7" fill="1" visible="no" active="yes"/>
+<layer number="199" name="Contour" color="7" fill="1" visible="no" active="yes"/>
 <layer number="200" name="200bmp" color="1" fill="10" visible="no" active="yes"/>
 <layer number="201" name="201bmp" color="2" fill="10" visible="no" active="yes"/>
@@
 </class>
 </classes>
-<designrules>
+<designrules name="default">
 <description language="de">&lt;b&gt;EAGLE Design Rules&lt;/b&gt;
 &lt;p&gt;
@@
 <element name="BAT1" library="SparkFun" package="BATTCON_20MM" value="cr2032" x="157.3" y="12.85"/>
 <element name="U$3" library="SparkFun" package="AVR_MINI_PROG" value="AVR_MINI_PROGSMD" x="128.09" y="16.66" rot="R180"/>
+<element name="Q1" library="transistor-fet" package="SC75_INFINEON" value="BSA223SP" x="2.54" y="-5.08"/>
 </elements>
 <signals>
@@
 <wire x1="157.3" y1="12.85" x2="153.9347" y2="12.85" width="0.254" layer="1"/>
 <wire x1="126.3882" y1="12.215" x2="127.8234" y2="12.215" width="0.254" layer="1"/>
+<contactref element="Q1" pad="1"/>
+<wire x1="2.04" y1="-5.655" x2="126.3882" y2="12.215" width="0" layer="19" extent="1-1"/>
+</signal>
+<signal name="RESET">
+<contactref element="U$1" pad="1"/>
+<contactref element="U$3" pad="3"/>
+<wire x1="124.953" y1="8.405" x2="124.4951" y2="8.8629" width="0.254" layer="1"/>
+<wire x1="124.4951" y1="8.8629" x2="124.4951" y2="8.9388" width="0.254" layer="1"/>
+<wire x1="125.09" y1="16.66" x2="125.09" y2="9.5337" width="0.254" layer="16"/>
+<wire x1="125.09" y1="9.5337" x2="124.4951" y2="8.9388" width="0.254" layer="16"/>
+<wire x1="126.3882" y1="8.405" x2="124.953" y2="8.405" width="0.254" layer="1"/>
+<via x="124.4951" y="8.9388" extent="1-16" drill="0.6096" diameter="1.016"/>
+</signal>
+<signal name="N$7">
+<contactref element="BAT1" pad="1"/>
 </signal>
 <signal name="2.8V">
-<contactref element="BAT1" pad="1"/>
+<contactref element="Q1" pad="3"/>
 <contactref element="U$1" pad="8"/>
 <contactref element="U$3" pad="1"/>
-<wire x1="144.8" y1="12.85" x2="141.4347" y2="12.85" width="0.254" layer="1"/>
 <wire x1="128.09" y1="16.66" x2="137.6247" y2="16.66" width="0.254" layer="1"/>
 <wire x1="137.6247" y1="16.66" x2="141.4347" y2="12.85" width="0.254" layer="1"/>
@@
 <wire x1="128.09" y1="15.6757" x2="128.0877" y2="15.6757" width="0.254" layer="16"/>
 <wire x1="128.0877" y1="15.6757" x2="126.2787" y2="13.8667" width="0.254" layer="16"/>
-</signal>
-<signal name="RESET">
-<contactref element="U$1" pad="1"/>
-<contactref element="U$3" pad="3"/>
-<wire x1="124.953" y1="8.405" x2="124.4951" y2="8.8629" width="0.254" layer="1"/>
-<wire x1="124.4951" y1="8.8629" x2="124.4951" y2="8.9388" width="0.254" layer="1"/>
-<wire x1="125.09" y1="16.66" x2="125.09" y2="9.5337" width="0.254" layer="16"/>
-<wire x1="125.09" y1="9.5337" x2="124.4951" y2="8.9388" width="0.254" layer="16"/>
-<wire x1="126.3882" y1="8.405" x2="124.953" y2="8.405" width="0.254" layer="1"/>
-<via x="124.4951" y="8.9388" extent="1-16" drill="0.6096" diameter="1.016"/>
+<wire x1="3.04" y1="-5.655" x2="119.6572" y2="8.405" width="0" layer="19" extent="1-1"/>
 </signal>
 </signals>
