File: Charlie/charlie heart.brd (EAGLE design)
At the start: 46.7 x 57.7 mm, 33 parts, among them Q1 BSS84

Commit message: remove pullup resistor
Parts:
- removed R6: 10k, rcl:R0805
Connections:
- net 2.8V: no longer R6.2
- net PB2/SCK: no longer R6.1
Routing:
- net N$4: track 23.6 -> 32.6 mm
- net PB2/SCK: track 33.7 -> 27.3 mm
- net 2.8V: track 28.2 -> 23.5 mm
- net N$3: track 51.9 -> 49.2 mm
- net N$6: track 26.9 -> 27.8 mm
